File: eagle/FanControl.brd (EAGLE design)
At the start: 11.4 x 24.4 mm, 18 parts, among them U1 LP2985

Commit message: Added extra pads for another 1-Wire device on the bottom layer.
Parts:
- added TP6, TP7, TP8: TPB1,27, testpad:B1,27
Connections:
- net 1WIRE: now also TP6.TP
- net 3.3V: now also TP8.TP
- net GND: now also TP7.TP
Routing:
- net GND: track 34.9 -> 52.1 mm, vias 1 -> 2
- net 3.3V: track 19.6 -> 22.2 mm, vias 0 -> 1
- net 1WIRE: track 10.6 -> 11.8 mm, vias 0 -> 1
Changed lines of the file:
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@@
 <text x="10.16" y="23.8125" size="1.778" layer="21" rot="R270">~</text>
 <text x="10.16" y="2.54" size="1.778" layer="21" rot="R270">~</text>
-<text x="10.795" y="16.8275" size="1.778" layer="21" rot="R180">~</text>
+<text x="10.795" y="19.05" size="1.778" layer="21" rot="R270">~</text>
 </plain>
 <attributes>
@@
 <attribute name="TP_SIGNAL_NAME" value="" x="7.62" y="17.145" size="1" layer="37"/>
 </element>
+<element name="TP6" library="testpad" package="B1,27" value="TPB1,27" x="9.8425" y="18.0975" smashed="yes" rot="MR0">
+<attribute name="TP_SIGNAL_NAME" value="" x="10.4775" y="16.1925" size="1" layer="38" rot="MR0"/>
+</element>
+<element name="TP7" library="testpad" package="B1,27" value="TPB1,27" x="9.8425" y="20.0025" smashed="yes" rot="MR0">
+<attribute name="TP_SIGNAL_NAME" value="" x="10.4775" y="18.0975" size="1" layer="38" rot="MR0"/>
+</element>
+<element name="TP8" library="testpad" package="B1,27" value="TPB1,27" x="8.255" y="19.05" smashed="yes" rot="MR0">
+<attribute name="TP_SIGNAL_NAME" value="" x="8.89" y="17.145" size="1" layer="38" rot="MR0"/>
+</element>
 </elements>
 <signals>
@@
 <wire x1="4.4196" y1="7.62" x2="3.81" y2="7.62" width="0.4064" layer="1"/>
 <wire x1="3.81" y1="7.62" x2="2.54" y2="8.89" width="0.4064" layer="1"/>
-<wire x1="2.54" y1="8.89" x2="1.27" y2="8.89" width="0.4064" layer="1"/>
-<wire x1="1.27" y1="8.89" x2="0.635" y2="9.525" width="0.4064" layer="1"/>
-<wire x1="0.635" y1="9.525" x2="0.635" y2="11.43" width="0.4064" layer="1"/>
+<wire x1="2.54" y1="8.89" x2="0.635" y2="8.89" width="0.4064" layer="1"/>
 <wire x1="0.635" y1="11.43" x2="1.905" y2="12.7" width="0.4064" layer="1"/>
 <wire x1="3.64" y1="20" x2="4.13" y2="20" width="0.4064" layer="1"/>
@@
 <wire x1="2.2225" y1="20.6375" x2="3.0025" y2="20.6375" width="0.8128" layer="1"/>
 <wire x1="3.0025" y1="20.6375" x2="3.64" y2="20" width="0.8128" layer="1"/>
+<contactref element="TP7" pad="TP"/>
+<wire x1="1.59" y1="4.445" x2="1.59" y2="3.1725" width="0.4064" layer="1"/>
+<wire x1="1.59" y1="3.1725" x2="3.175" y2="1.5875" width="0.4064" layer="1"/>
+<wire x1="7.5175" y1="4.445" x2="7.5175" y2="3.7075" width="0.4064" layer="1"/>
+<wire x1="7.5175" y1="3.7075" x2="6.985" y2="3.175" width="0.4064" layer="1"/>
+<wire x1="3.175" y1="1.5875" x2="4.7625" y2="3.175" width="0.4064" layer="1"/>
+<wire x1="4.7625" y1="3.175" x2="6.985" y2="3.175" width="0.4064" layer="1"/>
+<wire x1="1.59" y1="4.445" x2="1.59" y2="6.03" width="0.4064" layer="1"/>
+<wire x1="1.59" y1="6.03" x2="0.635" y2="6.985" width="0.4064" layer="1"/>
+<wire x1="0.635" y1="11.43" x2="0.635" y2="8.89" width="0.4064" layer="1"/>
+<wire x1="0.635" y1="8.89" x2="0.635" y2="6.985" width="0.4064" layer="1"/>
+<wire x1="9.8425" y1="20.0025" x2="9.8425" y2="21.2725" width="0.4064" layer="1"/>
+<via x="9.8425" y="21.2725" extent="1-16" drill="0.6"/>
+<wire x1="9.8425" y1="21.2725" x2="9.8425" y2="20.0025" width="0.4064" layer="16"/>
 </signal>
 <signal name="12V">
@@
 <contactref element="TP5" pad="TP"/>
 <wire x1="5.715" y1="18.1" x2="7.305" y2="18.1" width="0.4064" layer="1"/>
-<wire x1="7.305" y1="18.1" x2="8.255" y2="19.05" width="0.4064" layer="1"/>
+<contactref element="TP8" pad="TP"/>
+<wire x1="8.255" y1="19.05" x2="7.305" y2="18.1" width="0.4064" layer="1"/>
+<wire x1="8.255" y1="19.05" x2="8.255" y2="17.78" width="0.4064" layer="16"/>
+<via x="8.255" y="17.78" extent="1-16" drill="0.6"/>
+<wire x1="8.255" y1="17.78" x2="8.255" y2="19.05" width="0.4064" layer="1"/>
 </signal>
 <signal name="SIG">
@@
 <contactref element="U$4" pad="P$2"/>
 <wire x1="10.795" y1="13.97" x2="10.795" y2="15.875" width="0.4064" layer="1"/>
-<wire x1="10.795" y1="15.875" x2="10.16" y2="16.51" width="0.4064" layer="1"/>
 <wire x1="7.62" y1="16.51" x2="7.605" y2="16.51" width="0.4064" layer="1"/>
 <wire x1="7.605" y1="16.51" x2="6.985" y2="16.09" width="0.4064" layer="1"/>
@@
 <contactref element="TP1" pad="TP"/>
 <wire x1="9.8425" y1="16.51" x2="10.16" y2="16.51" width="0.4064" layer="1"/>
-<wire x1="9.8425" y1="18.0975" x2="9.8425" y2="16.51" width="0.4064" layer="1"/>
 <wire x1="10.795" y1="13.97" x2="9.525" y2="12.7" width="0.4064" layer="1"/>
+<contactref element="TP6" pad="TP"/>
+<via x="9.8425" y="16.8275" extent="1-16" drill="0.6"/>
+<wire x1="9.8425" y1="16.8275" x2="9.8425" y2="18.0975" width="0.4064" layer="16"/>
+<wire x1="10.16" y1="16.51" x2="10.795" y2="15.875" width="0.4064" layer="1"/>
+<wire x1="9.8425" y1="18.0975" x2="9.8425" y2="16.8275" width="0.4064" layer="1"/>
+<wire x1="9.8425" y1="16.8275" x2="9.8425" y2="16.51" width="0.4064" layer="1"/>
 </signal>
 <signal name="N$2">
